File: TopPlate/coconut42_TopPlate.kicad_pcb (KiCad board)
At the start: 2 copper layers, 230.6 x 90.2 mm, 18 parts

Commit message: v1.1: OLEDの電源を+3.3Vにするなど
Parts:
- removed the Ref** at (166.5, 99.2)
- removed the Ref** at (242.7, 61.1)
- removed the Ref** at (166.5, 61.1)
- removed the Ref** at (204.6, 99.2)
- removed the Ref** at (242.7, 80.1)
- removed rBT1, rBT2, rBT3, rBT4: Breakaway_Tabs, kbd:Breakaway_Tabs
- moved BT2 19.8 mm to (136.0, 41.8)
- moved BT3 19.6 mm to (59.8, 99.4)
- moved BT1 18.4 mm to (59.8, 41.8)
Other:
- board size 230.6 x 90.2 mm -> 114.3 x 90.2 mm
