File: PCB/coconut42.kicad_sch (KiCad schematic)
At the start: 220 parts, among them J1 OLED, J2 MJ-4PP-9, J3 OLED, J4 MJ-4PP-9, SW1 SW_PUSH, SW10 SW_PUSH, SW11 SW_PUSH, SW12 SW_PUSH, SW13 SW_PUSH, SW14 SW_PUSH, SW15 SW_PUSH, SW16 SW_PUSH, SW17 SW_PUSH, SW18 SW_PUSH, SW19 SW_PUSH, SW2 SW_PUSH, SW20 SW_PUSH, SW21 SW_PUSH, SW22 SW_PUSH, SW23 SW_PUSH, SW24 SW_PUSH, SW25 SW_PUSH, SW26 SW_PUSH, SW27 SW_PUSH, SW28 SW_PUSH, SW29 SW_PUSH, SW3 SW_PUSH, SW30 SW_PUSH, SW31 SW_PUSH, SW32 SW_PUSH, SW33 SW_PUSH, SW34 SW_PUSH, SW35 SW_PUSH, SW36 SW_PUSH, SW37 SW_PUSH, SW38 SW_PUSH, SW39 SW_PUSH, SW4 SW_PUSH, SW40 SW_PUSH, SW41 SW_PUSH, SW42 SW_PUSH, SW5 SW_PUSH, SW6 SW_PUSH, SW7 SW_PUSH, SW8 SW_PUSH, SW9 SW_PUSH, U1 MOUDLE-SEEEDUINO-XIAO, U2 MOUDLE-SEEEDUINO-XIAO

Commit message: v1.1: OLEDの電源を+3.3Vにするなど
Parts:
- removed C1, C2, C28, C29, C3, C30, C31, C32, C33, C4, C5, C55, C56, C6: 0.1u, kbd:C_0603_1608Metric_Pad1.08x0.95mm_HandSolder, symbol Device:C_Small
- LED1, LED2: footprint kbd:LED_WS2812B-PLCC4 -> LED_SMD:LED_WS2812B_PLCC4_5.0x5.0mm_P3.2mm
- SW1: value SW_PUSH -> [3, 0]
- SW10: value SW_PUSH -> [7, 2]
- SW11: value SW_PUSH -> [7, 1]
- SW12: value SW_PUSH -> [7, 0]
- SW13: value SW_PUSH -> [2, 0]
- SW14: value SW_PUSH -> [2, 1]
- SW15: value SW_PUSH -> [2, 3]
- SW16: value SW_PUSH -> [2, 4]
- SW17: value SW_PUSH -> [2, 5]
- SW18: value SW_PUSH -> [2, 6]
- SW19: value SW_PUSH -> [6, 6]
- SW2: value SW_PUSH -> [3, 1]
- SW20: value SW_PUSH -> [6, 5]
- SW21: value SW_PUSH -> [6, 4]
- SW22: value SW_PUSH -> [6, 3]
- SW23: value SW_PUSH -> [6, 1]
- SW24: value SW_PUSH -> [6, 0]
- SW25: value SW_PUSH -> [1, 0]
- SW26: value SW_PUSH -> [1, 2]
- SW27: value SW_PUSH -> [1, 3]
- SW28: value SW_PUSH -> [1, 4]
- SW29: value SW_PUSH -> [1, 5]
- SW3: value SW_PUSH -> [3, 2]
- SW30: value SW_PUSH -> [1, 6]
- SW31: value SW_PUSH -> [5, 6]
- SW32: value SW_PUSH -> [5, 5]
- SW33: value SW_PUSH -> [5, 4]
- SW34: value SW_PUSH -> [5, 3]
- SW35: value SW_PUSH -> [5, 2]
- SW36: value SW_PUSH -> [5, 0]
- SW37: value SW_PUSH -> [0, 4]
- SW38: value SW_PUSH -> [0, 5]
- SW39: value SW_PUSH -> [0, 6]
- SW4: value SW_PUSH -> [3, 4]
- SW40: value SW_PUSH -> [4, 6]
- SW41: value SW_PUSH -> [4, 5]
- SW42: value SW_PUSH -> [4, 4]
- SW5: value SW_PUSH -> [3, 5]
- SW6: value SW_PUSH -> [3, 6]
- SW7: value SW_PUSH -> [7, 6]
- SW8: value SW_PUSH -> [7, 5]
- SW9: value SW_PUSH -> [7, 4]
Connections:
- net 3V3: now also J1.3 (Pin_3), R2.2, R3.2; no longer R2.1, R3.1
- net 3V3_r: now also J3.3 (Pin_3), R7.2, R8.2; no longer R7.1, R8.1
- net P2: now also R2.1; no longer R2.2
- net P2_r: now also R7.1; no longer R7.2
- net VIN: no longer J1.3 (Pin_3)
- net VIN_r: no longer J3.3 (Pin_3)
- net data: now also R3.1; no longer R3.2
- net data_r: now also R8.1; no longer R8.2
Other:
- moved on the sheet: C52, C53, C54, D10, D11, D12, D19, D20, D21, D22, D23, D24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

Commit message: 名称を統一
Other:
- title: citron42 -> coconut42
Changed lines of the file:
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@@
 	(paper "A3")
 	(title_block
-		(title "citron42")
+		(title "coconut42")
 		(date "2024-08-16")
 		(rev "1.1")
